Commit message: Add Robotiq 2F-85 gripper option and UR tool communication
- robotiq-2f-85 gripper type using PickNik robotiq_description, mounted with
  the Robotiq coupling for UR e-series, with a grasp frame at the finger pads
- SRDF group, open/close states and collision macros for the 2F-85
- Controller config and spawning (activation controller on real hardware only)
- MoveIt gripper controller joints taken from the setup file
- Gazebo: add robotiq_description to GZ_SIM_RESOURCE_PATH when needed
- Per-arm tool communication (tool connector RS-485 as a local serial device),
  started from real.launch.py; the gripper uses it as its serial port
- Pass ur_type to ur_ros2_control, required since ur_robot_driver 3.9.0
- Add ros2_robotiq_gripper and serial to dependencies.repos

Co-Authored-By: Claude Opus 5.5 <noreply@anthropic.com>

File: prl_ur5_description/urdf/_gripper.urdf.xacro (robot description, xacro)
@@ -4,7 +4,7 @@
   <xacro:include filename="$(find onrobot_description)/urdf/onrobot_rg.urdf.xacro"/>
   <!-- Macro to generate gripper -->
-  <xacro:macro name="gripper" params="gripper prefix parent pose hardware_interface gz_sim">
+  <xacro:macro name="gripper" params="gripper prefix parent pose hardware_interface gz_sim com_port:=/dev/ttyUSB0">
     <!-- check gripper type -->
-    <xacro:unless value="${gripper in [None, 'onrobot-rg2', 'onrobot-rg6', 'onrobot-rg6-v2', 'weiss-wsg50'] or gripper.startswith('custom:') or gripper.startswith('allegro-hand:')}">
+    <xacro:unless value="${gripper in [None, 'onrobot-rg2', 'onrobot-rg6', 'onrobot-rg6-v2', 'weiss-wsg50', 'robotiq-2f-85'] or gripper.startswith('custom:') or gripper.startswith('allegro-hand:')}">
       <xacro:unknown_gripper_type/>
     </xacro:unless>
@@ -34,4 +34,23 @@
       </xacro:wsg_50_xacro>
     </xacro:if>
+    <!-- if robotiq-2f-85 -->
+    <xacro:if value="${gripper == 'robotiq-2f-85'}">
+      <xacro:include filename="$(find robotiq_description)/urdf/ur_to_robotiq_adapter.urdf.xacro"/>
+      <xacro:include filename="$(find robotiq_description)/urdf/robotiq_2f_85_macro.urdf.xacro"/>
+      <!-- Robotiq coupling for UR e-series flanges -->
+      <xacro:ur_to_robotiq prefix="${prefix}gripper_" parent="${parent}" child="${prefix}gripper_coupling"/>
+      <!-- Real hardware talks to the gripper over com_port (the UR tool connector or a USB adapter) -->
+      <xacro:robotiq_gripper name="${prefix}gripper" prefix="${prefix}gripper_" parent="${prefix}gripper_coupling"
+                             sim_gazebo="${gz_sim}" com_port="${com_port}">
+        <origin xyz="${pose['x']} ${pose['y']} ${pose['z']}" rpy="${pose['roll']} ${pose['pitch']} ${pose['yaw']}"/>
+      </xacro:robotiq_gripper>
+      <!-- Approximate centre of the finger pads; check against the real gripper -->
+      <link name="${prefix}gripper_grasp_frame"/>
+      <joint name="${prefix}gripper_grasp_frame_joint" type="fixed">
+        <parent link="${prefix}gripper_robotiq_85_base_link"/>
+        <child link="${prefix}gripper_grasp_frame"/>
+        <origin xyz="0 0 0.13" rpy="0 0 0"/>
+      </joint>
+    </xacro:if>
     <!-- if allegro-hand -->
     <xacro:if value="${gripper.startswith('allegro-hand:')}">

File: prl_ur5_description/urdf/mantis.urdf.xacro (robot description, xacro)
@@ -61,4 +61,7 @@
                  camera_pose="${left.get('camera_pose')}"
                  wrist_connector="${left.get('wrist_connector', True)}"
+                 tool_communication="${left.get('tool_communication', False)}"
+                 tool_device_name="${left.get('tool_device_name', '/tmp/ttyUR_left')}"
+                 gripper_com_port="${left.get('gripper_com_port', '/dev/ttyUSB0')}"
                  joint_limits_parameters_file="$(find prl_ur5_robot_configuration)/config/${left.get('arm_joint_limits')}"
                  kinematics_parameters_file="$(find prl_ur5_robot_configuration)/config/${left.get('arm_kinematics')}"
@@ -80,4 +83,7 @@
                  camera_pose="${right.get('camera_pose')}"
                  wrist_connector="${right.get('wrist_connector', True)}"
+                 tool_communication="${right.get('tool_communication', False)}"
+                 tool_device_name="${right.get('tool_device_name', '/tmp/ttyUR_right')}"
+                 gripper_com_port="${right.get('gripper_com_port', '/dev/ttyUSB0')}"
                  joint_limits_parameters_file="$(find prl_ur5_robot_configuration)/config/${right.get('arm_joint_limits')}"
                  kinematics_parameters_file="$(find prl_ur5_robot_configuration)/config/${right.get('arm_kinematics')}"

File: prl_ur5_description/urdf/ur5_complete_arm.urdf.xacro (robot description, xacro)
@@ -30,4 +30,7 @@
         visual_parameters_file:=''
         wrist_connector:=true
+        tool_communication:=false
+        tool_device_name:=/tmp/ttyUR
+        gripper_com_port:=/dev/ttyUSB0
         safety_limits:=false
         safety_pos_margin:=0.15
@@ -76,4 +79,8 @@
                 name="${prefix}arm"
                 tf_prefix="${prefix}"
+                ur_type="${ur_type}"
+                use_tool_communication="${tool_communication}"
+                tool_voltage="${24 if tool_communication else 0}"
+                tool_device_name="${tool_device_name}"
                 kinematics_parameters_file="${kinematics_parameters_file}"
                 robot_ip="${network['ip']}"
@@ -109,5 +116,7 @@
         </xacro:unless>
         <!-- Gripper -->
-        <xacro:gripper gripper="${gripper}" prefix='${prefix}' parent="${gripper_parent}" pose="${gripper_pose}" hardware_interface="${hw_interface}" gz_sim="${gz_sim}"/>
+        <!-- A gripper plugged into the tool connector is reached through the tool communication device -->
+        <xacro:property name="gripper_serial_port" value="${tool_device_name if tool_communication else gripper_com_port}"/>
+        <xacro:gripper gripper="${gripper}" prefix='${prefix}' parent="${gripper_parent}" pose="${gripper_pose}" hardware_interface="${hw_interface}" gz_sim="${gz_sim}" com_port="${gripper_serial_port}"/>
         <!-- Right angle connector -->
         <xacro:if value="${wrist_connector}">
