Commit message: Add selectable workcell with bimanual stand option
- Move the Vention table and walls into _workcell_mantis.urdf.xacro and add
  _workcell_bimanual_stand.urdf.xacro; select with the "workcell" key
  of the setup file (default "mantis", output unchanged)
- On the stand, arms are mounted on left/right_mount_plate and arm_pose is
  the offset from the plate
- Use the physical/visual parameters of "ur_type" (default "ur5")
- Make the Mantis wrist connector optional ("wrist_connector", default true)
- SRDF: keep the Mantis collision matrix for Mantis only; add a stand matrix
  that only disables rigidly attached pairs and keeps arm-to-arm checks
- SRDF: make fixed cameras optional, as in the URDF
- Fix setup file path being added to the active controllers in real.launch.py

Co-Authored-By: Claude Opus 5.5 <noreply@anthropic.com>

File: prl_ur5_description/urdf/mantis.urdf.xacro (robot description, xacro)
@@ -14,68 +14,35 @@
   <!-- Global frame -->
   <link name="prl_ur5_base"/>
-  <!-- Table -->
-  <material name="Blue">
-    <color rgba="${0/255} ${30/255} ${70/255} 1.0"/>
-  </material>
-  <link name="table_link">
-    <visual>
-      <geometry>
-        <mesh filename="file://$(find prl_ur5_description)/model/vention_table.stl"/>
-      </geometry>
-      <material name="Blue"/>
-    </visual>
-    <collision>
-      <geometry>
-        <mesh filename="file://$(find prl_ur5_description)/model/vention_table.stl"/>
-      </geometry>
-    </collision>
-  </link>
-  <joint name="table_fix" type="fixed">
-    <parent link="prl_ur5_base"/>
-    <child link = "table_link"/>
-    <origin xyz="0.0 0.0 0.0" rpy="0.0 0.0 0.0"/>
-  </joint>
+  <!-- Workcell: what the arms are mounted on (setup file key "workcell", default "mantis") -->
+  <xacro:include filename="$(find prl_ur5_description)/urdf/_workcell_mantis.urdf.xacro"/>
+  <xacro:include filename="$(find prl_ur5_description)/urdf/_workcell_bimanual_stand.urdf.xacro"/>
+  <xacro:property name="workcell" value="${setup_file.get('workcell', 'mantis')}"/>
+  <xacro:unless value="${workcell in ['mantis', 'bimanual_stand']}">
+    <xacro:unknown_workcell_type/>
+  </xacro:unless>
+  <!-- UR model used for the physical/visual parameters of both arms (default "ur5") -->
+  <xacro:property name="ur_type" value="${setup_file.get('ur_type', 'ur5')}"/>
+  <xacro:if value="${workcell == 'mantis'}">
+    <xacro:workcell_mantis parent="prl_ur5_base"/>
+    <!-- Height of the table top (prl_ur5_base) above the ground (base_link) -->
+    <xacro:property name="workcell_height" value="0.8"/>
+    <xacro:property name="left_arm_parent" value="prl_ur5_base"/>
+    <xacro:property name="right_arm_parent" value="prl_ur5_base"/>
+  </xacro:if>
+  <xacro:if value="${workcell == 'bimanual_stand'}">
+    <xacro:property name="stand" value="${setup_file.get('bimanual_stand') or dict()}"/>
+    <xacro:workcell_bimanual_stand parent="prl_ur5_base"
+      arm_mount_height="${stand.get('arm_mount_height', 1.5)}"
+      plate_position="${stand.get('plate_position', 0.0)}"/>
+    <!-- The stand origin is on the ground -->
+    <xacro:property name="workcell_height" value="0.0"/>
+    <!-- arm_pose of each arm is its offset from the mounting plate -->
+    <xacro:property name="left_arm_parent" value="left_mount_plate"/>
+    <xacro:property name="right_arm_parent" value="right_mount_plate"/>
+  </xacro:if>
   <!-- Cameras fixtures (if any) -->
   <xacro:if value="${setup_file.get('fixed_cameras_file') is not None}">
     <xacro:fixed_cameras parent="prl_ur5_base" fixed_cameras_file="$(find prl_ur5_robot_configuration)/config/${setup_file['fixed_cameras_file']}" turn_on="true"/>
   </xacro:if>
-  <!-- back wall -->
-  <link name="backwall_link">
-    <visual>
-      <geometry>
-        <box size="3.5 0.1 2" />
-      </geometry>
-      <material name="grey"><color rgba="0.8 0.8 0.8 0.2"/></material>
-    </visual>
-    <collision>
-      <geometry>
-        <box size="3.5 0.1 2" />
-      </geometry>
-    </collision>
-  </link>
-  <joint name="backwall_fix" type="fixed">
-    <parent link="prl_ur5_base"/>
-    <child link = "backwall_link"/>
-    <origin xyz="0 -1.05 0.25" rpy="0.0 0.0 0.0"/>
-  </joint>
-  <!-- left wall -->
-  <link name="leftwall_link">
-    <visual>
-      <geometry>
-        <box size="0.1 1.95 2" />
-      </geometry>
-      <material name="grey"><color rgba="0.8 0.8 0.8 0.1"/></material>
-    </visual>
-    <collision>
-      <geometry>
-        <box size="0.1 1.95 2" />
-      </geometry>
-    </collision>
-  </link>
-  <joint name="leftwall_fix" type="fixed">
-    <parent link="prl_ur5_base"/>
-    <child link = "leftwall_link"/>
-    <origin xyz="-1.65 0 0.25" rpy="0.0 0.0 0.0"/>
-  </joint>
   <!-- ARMS -->
   <!-- Left arm -->
@@ -83,5 +50,6 @@
   <xacro:property name="left_network" value="${network_file.get('left_network')}"/>
   <xacro:arm prefix="left_"
-                 parent="prl_ur5_base"
+                 parent="${left_arm_parent}"
+                 ur_type="${ur_type}"
                  pose="${left['arm_pose']}"
                  sensors="false"
@@ -92,4 +60,5 @@
                  camera="${left.get('camera')}"
                  camera_pose="${left.get('camera_pose')}"
+                 wrist_connector="${left.get('wrist_connector', True)}"
                  joint_limits_parameters_file="$(find prl_ur5_robot_configuration)/config/${left.get('arm_joint_limits')}"
                  kinematics_parameters_file="$(find prl_ur5_robot_configuration)/config/${left.get('arm_kinematics')}"
@@ -100,5 +69,6 @@
   <xacro:property name="right_network" value="${network_file.get('right_network')}"/>
   <xacro:arm prefix="right_"
-                 parent="prl_ur5_base"
+                 parent="${right_arm_parent}"
+                 ur_type="${ur_type}"
                  pose="${right['arm_pose']}"
                  sensors="false"
@@ -109,4 +79,5 @@
                  camera="${right.get('camera')}"
                  camera_pose="${right.get('camera_pose')}"
+                 wrist_connector="${right.get('wrist_connector', True)}"
                  joint_limits_parameters_file="$(find prl_ur5_robot_configuration)/config/${right.get('arm_joint_limits')}"
                  kinematics_parameters_file="$(find prl_ur5_robot_configuration)/config/${right.get('arm_kinematics')}"
@@ -126,5 +97,5 @@
     <parent link="base_link" />
     <child link="prl_ur5_base" />
-    <origin xyz="0 0 0.8" rpy="0 0 0" />
+    <origin xyz="0 0 ${workcell_height}" rpy="0 0 0" />
   </joint>
 </robot>

File: prl_ur5_description/urdf/ur5_complete_arm.urdf.xacro (robot description, xacro)
@@ -27,6 +27,7 @@
         kinematics_parameters_file:='$(find ur_description)/config/ur5/default_kinematics.yaml'
         hw_interface:=hardware_interface/PositionJointInterface
-        physical_parameters_file:='$(find ur_description)/config/ur5/physical_parameters.yaml'
-        visual_parameters_file:='$(find ur_description)/config/ur5/visual_parameters.yaml'
+        physical_parameters_file:=''
+        visual_parameters_file:=''
+        wrist_connector:=true
         safety_limits:=false
         safety_pos_margin:=0.15
@@ -39,4 +40,7 @@
         network := ''
         ">
+        <!-- Physical/visual parameters default to the ones of ur_type -->
+        <xacro:property name="ur_physical_parameters_file" value="${physical_parameters_file or '$(find ur_description)/config/' + ur_type + '/physical_parameters.yaml'}"/>
+        <xacro:property name="ur_visual_parameters_file" value="${visual_parameters_file or '$(find ur_description)/config/' + ur_type + '/visual_parameters.yaml'}"/>
         <!-- UR5 -->
         <xacro:ur_robot
@@ -46,6 +50,6 @@
             joint_limits_parameters_file="${joint_limits_parameters_file}"
             kinematics_parameters_file="${kinematics_parameters_file}"
-            physical_parameters_file="${physical_parameters_file}"
-            visual_parameters_file="${visual_parameters_file}"
+            physical_parameters_file="${ur_physical_parameters_file}"
+            visual_parameters_file="${ur_visual_parameters_file}"
             safety_limits="${safety_limits}"
             safety_pos_margin="${safety_pos_margin}"
@@ -107,22 +111,24 @@
         <xacro:gripper gripper="${gripper}" prefix='${prefix}' parent="${gripper_parent}" pose="${gripper_pose}" hardware_interface="${hw_interface}" gz_sim="${gz_sim}"/>
         <!-- Right angle connector -->
-        <link name="${prefix}wrist_connector_link">
-        <visual>
-            <geometry>
-                <mesh filename="file://$(find prl_ur5_description)/model/RG_connector_simple.stl"/>
-            </geometry>
-            <material name="connector_green"><color rgba="0.2 0.8 0 1"/></material>
-        </visual>
-        <collision>
-            <geometry>
-                <mesh filename="file://$(find prl_ur5_description)/model/RG_connector_simple_convex.stl"/>
-            </geometry>
-        </collision>
-        </link>
-        <joint name="${prefix}wrist_connector" type="fixed">
-        <origin xyz="0 -0.0375 -0.02" rpy="1.5708 0 0"/>
-        <parent link="${prefix}wrist_3_link"/>
-        <child link="${prefix}wrist_connector_link"/>
-        </joint>
+        <xacro:if value="${wrist_connector}">
+            <link name="${prefix}wrist_connector_link">
+            <visual>
+                <geometry>
+                    <mesh filename="file://$(find prl_ur5_description)/model/RG_connector_simple.stl"/>
+                </geometry>
+                <material name="connector_green"><color rgba="0.2 0.8 0 1"/></material>
+            </visual>
+            <collision>
+                <geometry>
+                    <mesh filename="file://$(find prl_ur5_description)/model/RG_connector_simple_convex.stl"/>
+                </geometry>
+            </collision>
+            </link>
+            <joint name="${prefix}wrist_connector" type="fixed">
+            <origin xyz="0 -0.0375 -0.02" rpy="1.5708 0 0"/>
+            <parent link="${prefix}wrist_3_link"/>
+            <child link="${prefix}wrist_connector_link"/>
+            </joint>
+        </xacro:if>
         <!-- hand-eye camera -->
         <xacro:unless value="${camera is None}">

Commit message: Fix the bimanual stand to the world in Gazebo
The stand links carry no mass and only rest on the ground plane, so the
cantilevered arms tipped the model over. The real stand is bolted down.

Co-Authored-By: Claude Opus 5.5 <noreply@anthropic.com>

File: prl_ur5_description/urdf/mantis.urdf.xacro (robot description, xacro)
@@ -107,3 +107,12 @@
     <origin xyz="0 0 ${workcell_height}" rpy="0 0 0" />
   </joint>
+  <!-- Gazebo: the stand is bolted to the floor. Without this it tips over under the cantilevered arms. -->
+  <xacro:if value="${workcell == 'bimanual_stand' and '$(arg gz_sim)'.lower() == 'true'}">
+    <link name="world"/>
+    <joint name="world_to_base_link" type="fixed">
+      <parent link="world"/>
+      <child link="base_link"/>
+      <origin xyz="0 0 0" rpy="0 0 0"/>
+    </joint>
+  </xacro:if>
 </robot>
