Commit message: Give the bimanual stand aluminium mass and optional anchoring
- Mass, centre of mass and inertia of the frame, brackets and plates computed
  from the meshes with aluminium (2700 kg/m3); brackets and plates are solid,
  the frame assumes 80x80 extrusion (40% of the solid mesh, 69.8 kg)
- frame_mass setting scales the frame inertia to a weighed value
- anchored setting (default true) to let the stand stand freely in Gazebo

Co-Authored-By: Claude Opus 5.5 <noreply@anthropic.com>

File: prl_ur5_description/urdf/_workcell_bimanual_stand.urdf.xacro (robot description, xacro)
@@ -4,6 +4,8 @@
        The frame origin is on the ground. Arms are mounted on left_mount_plate / right_mount_plate.
        arm_mount_height: height (m) from the ground to the top point of the angled bracket
-       plate_position:   plate position along the bracket (m); 0 = highest point, range roughly 0.0 to 0.12 -->
-  <xacro:macro name="workcell_bimanual_stand" params="parent arm_mount_height:=1.5 plate_position:=0.0">
+       plate_position:   plate position along the bracket (m); 0 = highest point, range roughly 0.0 to 0.12
+       frame_mass:       mass (kg) of the frame; the default assumes 80x80 aluminium extrusion (40% of the solid mesh)
+       Inertias were computed from the meshes with aluminium (2700 kg/m3); brackets and plates are solid. -->
+  <xacro:macro name="workcell_bimanual_stand" params="parent arm_mount_height:=1.5 plate_position:=0.0 frame_mass:=69.774">
     <xacro:property name="stand_mesh_dir" value="file://$(find prl_ur5_description)/model/bimanual_stand"/>
     <!-- Meshes are exported in cm -->
@@ -17,5 +19,13 @@
       <color rgba="0.5 0.5 0.5 1.0"/>
     </material>
+    <!-- Frame inertia scales with frame_mass (69.774 kg at 40% fill) -->
+    <xacro:property name="frame_inertia_scale" value="${frame_mass / 69.774}"/>
     <link name="stand_frame">
+      <inertial>
+        <origin xyz="-0.1294 0.0001 0.5820" rpy="0 0 0"/>
+        <mass value="${frame_mass}"/>
+        <inertia ixx="${19.86539 * frame_inertia_scale}" ixy="${-0.00215 * frame_inertia_scale}" ixz="${2.43733 * frame_inertia_scale}"
+                 iyy="${18.28416 * frame_inertia_scale}" iyz="${0.00446 * frame_inertia_scale}" izz="${6.19608 * frame_inertia_scale}"/>
+      </inertial>
       <visual>
         <geometry>
@@ -37,6 +47,12 @@
     </joint>
     <!-- Angled bracket + mounting plate for one arm -->
-    <xacro:macro name="bimanual_stand_arm_mount" params="prefix mount_xyz mount_rpy bracket_mesh plate_xyz">
+    <xacro:macro name="bimanual_stand_arm_mount" params="prefix mount_xyz mount_rpy bracket_mesh plate_xyz bracket_side">
       <link name="${prefix}mount_assembly">
+        <!-- Solid aluminium bracket; bracket_side mirrors the COM and iyz for the two brackets -->
+        <inertial>
+          <origin xyz="0 ${0.0417 * bracket_side} 0.0417" rpy="0 0 0"/>
+          <mass value="8.449"/>
+          <inertia ixx="0.10653" ixy="0" ixz="0" iyy="0.08474" iyz="${0.02800 * bracket_side}" izz="0.08487"/>
+        </inertial>
         <visual>
           <geometry>
@@ -58,4 +74,9 @@
       </joint>
       <link name="${prefix}mount_plate">
+        <!-- Solid aluminium plate, 160 x 160 x 20 mm -->
+        <inertial>
+          <mass value="1.382"/>
+          <inertia ixx="0.00300" ixy="0" ixz="0" iyy="0.00300" iyz="0" izz="0.00590"/>
+        </inertial>
         <visual>
           <geometry>
@@ -78,8 +99,8 @@
     <xacro:bimanual_stand_arm_mount prefix="left_"
       mount_xyz="-0.212 0.2754 ${mount_z}" mount_rpy="${radians(-45)} 0 0"
-      bracket_mesh="angled_arm_2.stl" plate_xyz="0 ${-plate_y} 0.14953"/>
+      bracket_mesh="angled_arm_2.stl" plate_xyz="0 ${-plate_y} 0.14953" bracket_side="1"/>
     <xacro:bimanual_stand_arm_mount prefix="right_"
       mount_xyz="-0.212 -0.2754 ${mount_z}" mount_rpy="${radians(45)} 0 0"
-      bracket_mesh="angled_arm_1.stl" plate_xyz="0 ${plate_y} 0.14953"/>
+      bracket_mesh="angled_arm_1.stl" plate_xyz="0 ${plate_y} 0.14953" bracket_side="-1"/>
   </xacro:macro>
 </robot>

File: prl_ur5_description/urdf/mantis.urdf.xacro (robot description, xacro)
@@ -34,5 +34,6 @@
     <xacro:workcell_bimanual_stand parent="prl_ur5_base"
       arm_mount_height="${stand.get('arm_mount_height', 1.5)}"
-      plate_position="${stand.get('plate_position', 0.0)}"/>
+      plate_position="${stand.get('plate_position', 0.0)}"
+      frame_mass="${stand.get('frame_mass', 69.774)}"/>
     <!-- The stand origin is on the ground -->
     <xacro:property name="workcell_height" value="0.0"/>
@@ -107,6 +108,6 @@
     <origin xyz="0 0 ${workcell_height}" rpy="0 0 0" />
   </joint>
-  <!-- Gazebo: the stand is bolted to the floor. Without this it tips over under the cantilevered arms. -->
-  <xacro:if value="${workcell == 'bimanual_stand' and '$(arg gz_sim)'.lower() == 'true'}">
+  <!-- Gazebo: the stand is bolted to the floor. Set "anchored: false" to let it stand freely on its casters. -->
+  <xacro:if value="${workcell == 'bimanual_stand' and stand.get('anchored', True) and '$(arg gz_sim)'.lower() == 'true'}">
     <link name="world"/>
     <joint name="world_to_base_link" type="fixed">
