Commit message: Add ZED Mini / ZED 2i cameras and fix wrist cameras
- zed-mini and zed-2i camera types (zed_description), for wrist and fixed
  cameras, with generic Gazebo colour and depth sensors named like the D435 ones
- Wrist cameras are mounted where the gripper is (tool0 or the F/T sensor tool
  frame) instead of the F/T sensor frame only, and are on in Gazebo
- Fixed cameras: "fixture: none" to skip the Mantis camera post
- SRDF: fixture pairs only with the post; ZED wrist camera pairs with its
  gripper and wrist 3
- Camera config file of the setup ("cameras_config_file") used by
  sensors.launch.py, the Gazebo camera bridge and depth alignment
- Gazebo camera bridge generated at launch from the camera config (the static
  one listed cameras that are no longer configured)
- Gazebo resource path for robotiq, zed and realsense description meshes
- Add zed-ros2-description to dependencies.repos

Co-Authored-By: Claude Opus 5.5 <noreply@anthropic.com>

File: prl_ur5_description/urdf/_camera_sensor.urdf.xacro (robot description, xacro)
@@ -6,5 +6,5 @@
   <xacro:macro name="camera_sensor" params="prefix parent camera pose turn_on:=false">
     <!-- check camera type -->
-    <xacro:unless value="${camera in ['realsense-d435i', 'femto-mega', None]}">
+    <xacro:unless value="${camera in ['realsense-d435i', 'femto-mega', 'zed-mini', 'zed-2i', None]}">
       <xacro:unknown_camera_type/>
     </xacro:unless>
@@ -16,4 +16,10 @@
       <xacro:gazebo_d435 name="${prefix}camera" turn_on="${turn_on}"/>
     </xacro:if>
+    <!-- if Stereolabs ZED Mini / ZED 2i (pose is the pose of the camera's mounting screw) -->
+    <xacro:if value="${camera in ['zed-mini', 'zed-2i']}">
+      <xacro:include filename="$(find prl_ur5_description)/urdf/_zed.urdf.xacro"/>
+      <xacro:zed_sensor name="${prefix}camera" model="${'zedm' if camera == 'zed-mini' else 'zed2i'}"
+                        parent="${parent}" pose="${pose}" turn_on="${turn_on}"/>
+    </xacro:if>
     <xacro:if value="${camera == 'femto-mega'}">
         <xacro:femto_bolt prefix="${prefix}camera" parent="${parent}" use_nominal_extrinsics="true">

File: prl_ur5_description/urdf/_fixed_cameras.urdf.xacro (robot description, xacro)
@@ -24,5 +24,5 @@
         <!-- Spawn camera -->
         <!-- check camera type -->
-        <xacro:unless value="${camera['type'] in ['realsense-d435i', 'femto-mega', 'None']}">
+        <xacro:unless value="${camera['type'] in ['realsense-d435i', 'femto-mega', 'zed-mini', 'zed-2i', 'None']}">
             <xacro:unknown_camera_type/>
         </xacro:unless>
@@ -57,112 +57,124 @@
                                 pose="${dict(x=-0.0307, y=0.02014, z=-0.03425, roll=pi/2.0, pitch=-pi/2.0, yaw=0.0)}" />
         </xacro:if>
-        <!-- Numerical dimensions for the fixtures -->
-        <xacro:property name="extrusion_width" value="${0.045 +0.06}"/> <!-- +/-3cm margin on the real size -->
-        <xacro:property name="hr_z_pos_absolute" value="-0.05625"/> <!-- height at which the horizontal extrusion are fixed to the table -->
-        <xacro:property name="sj_height" value="${0.08 + 0.09}"/> <!-- Height of the spherical joint supporting the camera + the angle piece supporting the spherical joint -->
-        <xacro:property name="sj_diameter" value="${0.09 +0.03}"/> <!-- Diameter of the spherical joint supporting the camera -->
-        <!-- Simple math to change the side of the table to which the fixture is attached-->
-        <!-- The arbitrary values 0.92 0.92 0.29 0.52 correspond to the dimensions of the table with 1cm margin, so the extrusions are not touching the table-->
-        <xacro:if value="${camera['fixture_orientation'] == '+x'}">
-            <xacro:property name="hr_len" value="${camera['pose']['x'] - camera['offset']['x'] + extrusion_width/2. - 0.92}"/>
-            <xacro:property name="hr_x_pos_relative" value="${- hr_len/2. + extrusion_width/2.}"/>
-            <xacro:property name="hr_y_pos_relative" value="0"/>
-            <xacro:property name="hr_z_rot_relative" value="0"/>
+        <!-- if Stereolabs ZED: pose is the pose of the camera's mounting screw -->
+        <xacro:if value="${camera['type'] in ['zed-mini', 'zed-2i']}">
+            <xacro:camera_sensor camera="${camera['type']}"
+                                 prefix="${camera['name_prefix']}_"
+                                 parent="${parent}"
+                                 turn_on="${turn_on}"
+                                 pose="${camera['pose']}"/>
         </xacro:if>
-        <xacro:if value="${camera['fixture_orientation'] == '-x'}">
-            <xacro:property name="hr_len" value="${-camera['pose']['x'] + camera['offset']['x'] + extrusion_width/2. - 0.92}"/>
-            <xacro:property name="hr_x_pos_relative" value="${hr_len/2. - extrusion_width/2.}"/>
-            <xacro:property name="hr_y_pos_relative" value="0"/>
-            <xacro:property name="hr_z_rot_relative" value="3.1415926"/>
+        <!-- Mantis camera post (extrusions fixed to the table). Set "fixture: none" for a camera on a tripod
+             or any mount that is not modelled. -->
+        <xacro:if value="${camera.get('fixture', 'mantis_post') != 'none'}">
+            <!-- Numerical dimensions for the fixtures -->
+            <xacro:property name="extrusion_width" value="${0.045 +0.06}"/> <!-- +/-3cm margin on the real size -->
+            <xacro:property name="hr_z_pos_absolute" value="-0.05625"/> <!-- height at which the horizontal extrusion are fixed to the table -->
+            <xacro:property name="sj_height" value="${0.08 + 0.09}"/> <!-- Height of the spherical joint supporting the camera + the angle piece supporting the spherical joint -->
+            <xacro:property name="sj_diameter" value="${0.09 +0.03}"/> <!-- Diameter of the spherical joint supporting the camera -->
+            <!-- Simple math to change the side of the table to which the fixture is attached-->
+            <!-- The arbitrary values 0.92 0.92 0.29 0.52 correspond to the dimensions of the table with 1cm margin, so the extrusions are not touching the table-->
+            <xacro:if value="${camera['fixture_orientation'] == '+x'}">
+                <xacro:property name="hr_len" value="${camera['pose']['x'] - camera['offset']['x'] + extrusion_width/2. - 0.92}"/>
+                <xacro:property name="hr_x_pos_relative" value="${- hr_len/2. + extrusion_width/2.}"/>
+                <xacro:property name="hr_y_pos_relative" value="0"/>
+                <xacro:property name="hr_z_rot_relative" value="0"/>
+            </xacro:if>
+            <xacro:if value="${camera['fixture_orientation'] == '-x'}">
+                <xacro:property name="hr_len" value="${-camera['pose']['x'] + camera['offset']['x'] + extrusion_width/2. - 0.92}"/>
+                <xacro:property name="hr_x_pos_relative" value="${hr_len/2. - extrusion_width/2.}"/>
+                <xacro:property name="hr_y_pos_relative" value="0"/>
+                <xacro:property name="hr_z_rot_relative" value="3.1415926"/>
+            </xacro:if>
+            <xacro:if value="${camera['fixture_orientation'] == '+y'}">
+                <xacro:property name="hr_len" value="${camera['pose']['y'] - camera['offset']['y'] + extrusion_width/2.  - 0.29}"/>
+                <xacro:property name="hr_x_pos_relative" value="0"/>
+                <xacro:property name="hr_y_pos_relative" value="${- hr_len/2. + extrusion_width/2.}"/>
+                <xacro:property name="hr_z_rot_relative" value="1.570796327"/>
+            </xacro:if>
+            <xacro:if value="${camera['fixture_orientation'] == '-y'}">
+                <xacro:property name="hr_len" value="${-camera['pose']['y'] + camera['offset']['y'] + extrusion_width/2.  - 0.52}"/>
+                <xacro:property name="hr_x_pos_relative" value="0"/>
+                <xacro:property name="hr_y_pos_relative" value="${hr_len/2. - extrusion_width/2.}"/>
+                <xacro:property name="hr_z_rot_relative" value="-1.570796327"/>
+            </xacro:if>
+            <xacro:property name="vt_len" value="${camera['pose']['z'] - camera['offset']['z'] - hr_z_pos_absolute}"/>
+            <!-- Camera bounding box -->
+            <link name="fixed_camera_${number}_bb">
+                <visual>
+                    <geometry>
+                        <cylinder radius="${camera['bounding_box']['width']/2.}" length="${camera['bounding_box']['height']}"/>
+                    </geometry>
+                    <material name="purple"><color rgba="0.01 0.32 0.41 0.1"/></material>
+                </visual>
+                <collision>
+                    <geometry>
+                        <cylinder radius="${camera['bounding_box']['width']/2.}" length="${camera['bounding_box']['height']}"/>
+                    </geometry>
+                </collision>
+            </link>
+            <joint name="fixed_camera_${number}_bb_joint" type="fixed">
+                <parent link = "${parent}"/>
+                <child link="fixed_camera_${number}_bb"/>
+                <origin xyz="${camera['pose']['x']} ${camera['pose']['y']} ${camera['pose']['z']}" rpy="0 0 0"/>
+            </joint>
+            <!-- Spherical joint holding the camera -->
+            <link name="fixed_camera_${number}_sj">
+                <visual>
+                    <geometry>
+                        <cylinder radius="${sj_diameter/2}" length="${sj_height}"/>
+                    </geometry>
+                    <material name="purple"/>
+                </visual>
+                <collision>
+                    <geometry>
+                        <cylinder radius="${sj_diameter/2}" length="${sj_height}"/>
+                    </geometry>
+                </collision>
+            </link>
+            <joint name="fixed_camera_${number}_sj_joint" type="fixed">
+                <parent link = "fixed_camera_${number}_bb"/>
+                <child link="fixed_camera_${number}_sj"/>
+                <origin xyz="0 0 ${- camera['bounding_box']['height']/2. - sj_height/2.}" rpy="0 0 0"/>
+            </joint>
+            <!-- Vertical extrusion -->
+            <link name="fixed_camera_${number}_vt">
+                <visual>
+                    <geometry>
+                        <box size="${extrusion_width} ${extrusion_width} ${vt_len}" />
+                    </geometry>
+                    <material name="purple"/>
+                </visual>
+                <collision>
+                    <geometry>
+                        <box size="${extrusion_width} ${extrusion_width} ${vt_len}" />
+                    </geometry>
+                </collision>
+            </link>
+            <joint name="fixed_camera_${number}_vt_joint" type="fixed">
+                <parent link = "fixed_camera_${number}_sj"/>
+                <child link="fixed_camera_${number}_vt"/>
+                <origin xyz="${-camera['offset']['x']} ${-camera['offset']['y']} ${sj_height/2. + camera['bounding_box']['height']/2. - camera['offset']['z'] - vt_len/2.}" rpy="0 0 0"/>
+            </joint>
+            <!-- Horizontal extrusion -->
+            <link name="fixed_hr_${number}">
+                <visual>
+                    <geometry>
+                        <box size="${hr_len} ${extrusion_width} ${extrusion_width}" />
+                    </geometry>
+                    <material name="purple"/>
+                </visual>
+                <collision>
+                    <geometry>
+                        <box size="${hr_len} ${extrusion_width} ${extrusion_width}" />
+                    </geometry>
+                </collision>
+            </link>
+            <joint name="fixed_hr_${number}_fix" type="fixed">
+                <parent link = "fixed_camera_${number}_vt"/>
+                <child link="fixed_hr_${number}"/>
+                <origin xyz="${hr_x_pos_relative} ${hr_y_pos_relative} ${- vt_len/2. - extrusion_width/2.}" rpy="0 0 ${hr_z_rot_relative}"/>
+            </joint>
         </xacro:if>
-        <xacro:if value="${camera['fixture_orientation'] == '+y'}">
-            <xacro:property name="hr_len" value="${camera['pose']['y'] - camera['offset']['y'] + extrusion_width/2.  - 0.29}"/>
-            <xacro:property name="hr_x_pos_relative" value="0"/>
-            <xacro:property name="hr_y_pos_relative" value="${- hr_len/2. + extrusion_width/2.}"/>
-            <xacro:property name="hr_z_rot_relative" value="1.570796327"/>
-        </xacro:if>
-        <xacro:if value="${camera['fixture_orientation'] == '-y'}">
-            <xacro:property name="hr_len" value="${-camera['pose']['y'] + camera['offset']['y'] + extrusion_width/2.  - 0.52}"/>
-            <xacro:property name="hr_x_pos_relative" value="0"/>
-            <xacro:property name="hr_y_pos_relative" value="${hr_len/2. - extrusion_width/2.}"/>
-            <xacro:property name="hr_z_rot_relative" value="-1.570796327"/>
-        </xacro:if>
-        <xacro:property name="vt_len" value="${camera['pose']['z'] - camera['offset']['z'] - hr_z_pos_absolute}"/>
-        <!-- Camera bounding box -->
-        <link name="fixed_camera_${number}_bb">
-            <visual>
-                <geometry>
-                    <cylinder radius="${camera['bounding_box']['width']/2.}" length="${camera['bounding_box']['height']}"/>
-                </geometry>
-                <material name="purple"><color rgba="0.01 0.32 0.41 0.1"/></material>
-            </visual>
-            <collision>
-                <geometry>
-                    <cylinder radius="${camera['bounding_box']['width']/2.}" length="${camera['bounding_box']['height']}"/>
-                </geometry>
-            </collision>
-        </link>
-        <joint name="fixed_camera_${number}_bb_joint" type="fixed">
-            <parent link = "${parent}"/>
-            <child link="fixed_camera_${number}_bb"/>
-            <origin xyz="${camera['pose']['x']} ${camera['pose']['y']} ${camera['pose']['z']}" rpy="0 0 0"/>
-        </joint>
-        <!-- Spherical joint holding the camera -->
-        <link name="fixed_camera_${number}_sj">
-            <visual>
-                <geometry>
-                    <cylinder radius="${sj_diameter/2}" length="${sj_height}"/>
-                </geometry>
-                <material name="purple"/>
-            </visual>
-            <collision>
-                <geometry>
-                    <cylinder radius="${sj_diameter/2}" length="${sj_height}"/>
-                </geometry>
-            </collision>
-        </link>
-        <joint name="fixed_camera_${number}_sj_joint" type="fixed">
-            <parent link = "fixed_camera_${number}_bb"/>
-            <child link="fixed_camera_${number}_sj"/>
-            <origin xyz="0 0 ${- camera['bounding_box']['height']/2. - sj_height/2.}" rpy="0 0 0"/>
-        </joint>
-        <!-- Vertical extrusion -->
-        <link name="fixed_camera_${number}_vt">
-            <visual>
-                <geometry>
-                    <box size="${extrusion_width} ${extrusion_width} ${vt_len}" />
-                </geometry>
-                <material name="purple"/>
-            </visual>
-            <collision>
-                <geometry>
-                    <box size="${extrusion_width} ${extrusion_width} ${vt_len}" />
-                </geometry>
-            </collision>
-        </link>
-        <joint name="fixed_camera_${number}_vt_joint" type="fixed">
-            <parent link = "fixed_camera_${number}_sj"/>
-            <child link="fixed_camera_${number}_vt"/>
-            <origin xyz="${-camera['offset']['x']} ${-camera['offset']['y']} ${sj_height/2. + camera['bounding_box']['height']/2. - camera['offset']['z'] - vt_len/2.}" rpy="0 0 0"/>
-        </joint>
-        <!-- Horizontal extrusion -->
-        <link name="fixed_hr_${number}">
-            <visual>
-                <geometry>
-                    <box size="${hr_len} ${extrusion_width} ${extrusion_width}" />
-                </geometry>
-                <material name="purple"/>
-            </visual>
-            <collision>
-                <geometry>
-                    <box size="${hr_len} ${extrusion_width} ${extrusion_width}" />
-                </geometry>
-            </collision>
-        </link>
-        <joint name="fixed_hr_${number}_fix" type="fixed">
-            <parent link = "fixed_camera_${number}_vt"/>
-            <child link="fixed_hr_${number}"/>
-            <origin xyz="${hr_x_pos_relative} ${hr_y_pos_relative} ${- vt_len/2. - extrusion_width/2.}" rpy="0 0 ${hr_z_rot_relative}"/>
-        </joint>
     </xacro:macro>
 </robot>

File: prl_ur5_description/urdf/ur5_complete_arm.urdf.xacro (robot description, xacro)
@@ -170,5 +170,6 @@
         <!-- hand-eye camera -->
         <xacro:unless value="${camera is None}">
-            <xacro:camera_sensor camera="${camera}" prefix='${prefix}' parent="${prefix}tool" pose="${camera_pose}" turn_on="${sensors}"/>
+            <!-- Mounted where the gripper is mounted (tool0, or the F/T sensor tool frame); always on in Gazebo -->
+            <xacro:camera_sensor camera="${camera}" prefix='${prefix}' parent="${gripper_parent}" pose="${camera_pose}" turn_on="${sensors in [True, 'true', 'True'] or gz_sim in [True, 'true', 'True']}"/>
         </xacro:unless>
     </xacro:macro>
